File: pcb/ProyectoFinalRougier_v1/ProyectoFinalRougier.sch (KiCad schematic (older format))
At the start: 28 parts, among them J1 Screw_Terminal_01x02, J2 Conn_01x06, J3 Screw_Terminal_01x02, U1 AD8495, U2 TL431DBZ, U3 AD8495, U4 TL431DBZ

Commit message: Se agregan 2 carpetas con el mismo proyecto pero con distinta disposición del PCB.
Parts:
- J1: Mouser Cod: (none) -> 651-1888807
- J2: renamed from J3; Mouser Cod: (none) -> 651-1888807
- U1: Mouser Cod: (none) -> 584-AD8495ARMZ-R7
- U2: renamed from U3; Mouser Cod: (none) -> 584-AD8495ARMZ-R7
- U3: renamed from U2; Mouser Cod: (none) -> 595-TL431BIDBZR
- U4: Mouser Cod: (none) -> 595-TL431BIDBZR
- renumbered C2 to C1, C3 to C2, C4 to C3, C6 to C4, C7 to C5, C8 to C6, C1 to C7, C5 to C8, J2 to J3, R5 to R4, R6 to R5, R7 to R6, R4 to R7
Connections:
- net at R3.1: now also J1.1 (Pin_1); no longer J1.2 (Pin_2)
- net at R1.1, R2.1: now also J1.2 (Pin_2); no longer J1.1 (Pin_1)
- net at R6.1: now also J2.1 (Pin_1); no longer J2.2 (Pin_2)
- net at R4.1, R5.1: now also J2.2 (Pin_2); no longer J2.1 (Pin_1)
Other:
- note added: "1 - 5V"
- note added: "2 - GND"
- note added: "3 - T1+"
- note added: "4 - T1(GND)"
- note added: "5 - T2+"
- note added: "6 - T2(GND)"
- note added: "Termocupla 1"
- note added: "Termocupla 2"
- moved on the sheet: J3, R4
